Commit message: Added rb1 robot model visuals/collisions/inertias and display launch file for rviz2

File: my_rb1_description/urdf/my_rb1_robot.urdf (robot description, URDF)
Before this commit: robot robot, 2 links, 1 joints
Links:
- added link back_caster, mass 0.5; collision sphere radius=0.025; visual sphere radius=0.025
- added link front_caster, mass 0.5; collision sphere radius=0.025; visual sphere radius=0.025
- added link front_laser
- added link left_wheel, mass 1.5; collision cylinder length=0.025 radius=0.025; visual cylinder length=0.025 radius=0.025
- added link right_wheel, mass 1.5; collision cylinder length=0.025 radius=0.025; visual cylinder length=0.025 radius=0.025
- link base_link: mass None -> 21
Joints:
- added joint base_link_back_caster_joint: type fixed, parent base_link, child back_caster, origin xyz=-0.1 0.0 -0.15 rpy=0 0 0
- added joint base_link_front_caster_joint: type fixed, parent base_link, child front_caster, origin xyz=0.1 0.0 -0.15 rpy=0 0 0
- added joint base_link_front_laser_joint: type fixed, parent base_link, child front_laser, origin xyz=0.25 0.0 0.075 rpy=3.141 0 0
- added joint base_link_left_wheel_joint: type continuous, parent base_link, child left_wheel, origin xyz=0 0.2 -0.15 rpy=0 0 0, axis 0 1 0, limit effort=10000 velocity=1000
- added joint base_link_right_wheel_joint: type continuous, parent base_link, child right_wheel, origin xyz=0 -0.2 -0.15 rpy=0 0 0, axis 0 1 0, limit effort=10000 velocity=1000
